Commit message: -Fix plate collision geometries resulting in buggy LIDAR simulation in Gazebo on Hydro by removing them

File: turtlebot_description/urdf/stacks/circles.urdf.xacro (robot description, xacro)
@@ -166,7 +166,8 @@
       </visual>
       <collision>
-        <origin xyz="0.0 0.0 0.0" rpy="0 0 0" />
-        <geometry>
-          <box size="0.233502 0.314845 0.006401"/>
+        <origin xyz="0.1 0.0 0.0" rpy="0 0 0" />
+        <geometry>
+          <!--<box size="0.233502 0.314845 0.006401"/>-->
+          <!--<cylinder length="0.006401" radius="0.15"/>-->
         </geometry>
       </collision>
@@ -198,5 +199,5 @@
         <origin xyz="0.0 0.0 0.0" rpy="0 0 0" />
         <geometry>
-          <box size="0.314856 0.314856 0.006401"/>
+          <!--<box size="0.314856 0.314856 0.006401"/>-->
         </geometry>
       </collision>
@@ -228,5 +229,5 @@
         <origin xyz="0.0 0.0 0.0" rpy="0 0 0" />
         <geometry>
-          <box size="0.314856 0.314856 0.006401"/>
+          <!--<box size="0.314856 0.314856 0.006401"/>-->
         </geometry>
       </collision>
@@ -260,5 +261,5 @@
         <origin xyz="0.0 0.0 0.0" rpy="0 0 0" />
         <geometry>
-          <box size="0.288 0.315 0.006401"/>
+          <!--<box size="0.288 0.315 0.006401"/>-->
         </geometry>
       </collision>

Commit message: -Comment out full collision geom tag so we don´t get warnings about empty collision tags when starting gazebo

File: turtlebot_description/urdf/stacks/circles.urdf.xacro (robot description, xacro)
@@ -165,11 +165,12 @@
         </geometry>
       </visual>
-      <collision>
-        <origin xyz="0.1 0.0 0.0" rpy="0 0 0" />
-        <geometry>
-          <!--<box size="0.233502 0.314845 0.006401"/>-->
-          <!--<cylinder length="0.006401" radius="0.15"/>-->
-        </geometry>
-      </collision>
+      <!--
+      <collision>
+        <origin xyz="0.0 0.0 0.0" rpy="0 0 0" />
+        <geometry>
+          <box size="0.233502 0.314845 0.006401"/>
+        </geometry>
+      </collision>
+      -->
     </link>
     <turtlebot_standoff_2in parent="${parent}" number="0" x_loc="0.0676402" y_loc="0.1314196" z_loc="0.0709803"/>
@@ -196,10 +197,12 @@
         </geometry>
       </visual>
-      <collision>
-        <origin xyz="0.0 0.0 0.0" rpy="0 0 0" />
-        <geometry>
-          <!--<box size="0.314856 0.314856 0.006401"/>-->
-        </geometry>
-      </collision>
+      <!--
+      <collision>
+        <origin xyz="0.0 0.0 0.0" rpy="0 0 0" />
+        <geometry>
+          <box size="0.314856 0.314856 0.006401"/>
+        </geometry>
+      </collision>
+      -->
     </link>
     <turtlebot_standoff_2in parent="standoff_2in_0_link" number="4" x_loc="0" y_loc="0" z_loc="0.05715"/>
@@ -226,10 +229,12 @@
         </geometry>
       </visual>
-      <collision>
-        <origin xyz="0.0 0.0 0.0" rpy="0 0 0" />
-        <geometry>
-          <!--<box size="0.314856 0.314856 0.006401"/>-->
-        </geometry>
-      </collision>
+      <!--
+      <collision>
+        <origin xyz="0.0 0.0 0.0" rpy="0 0 0" />
+        <geometry>
+          <box size="0.314856 0.314856 0.006401"/>
+        </geometry>
+      </collision>
+      -->
     </link>
     <turtlebot_standoff_kinect parent="plate_2_link" number="0" x_loc="-0.1024382" y_loc="0.098" z_loc="0.0032004"/>
@@ -258,10 +263,12 @@
         </geometry>
       </visual>
-      <collision>
-        <origin xyz="0.0 0.0 0.0" rpy="0 0 0" />
-        <geometry>
-          <!--<box size="0.288 0.315 0.006401"/>-->
-        </geometry>
-      </collision>
+      <!--
+      <collision>
+        <origin xyz="0.0 0.0 0.0" rpy="0 0 0" />
+        <geometry>
+          <box size="0.288 0.315 0.006401"/>
+        </geometry>
+      </collision>
+      -->
     </link>
   </xacro:macro>
